File: Design_Proposal/Power_SubModule/power.kicad_sch (KiCad schematic)
At the start: 22 parts, among them IC1 DW01A-G, J5 Header-Male-2.54_1x6, J6 MICROXNJ, J7 Header-Male-2.54_1x6, J8 TP4056, Q1 FS8205A, U3 AMS1117-3.3

Commit message: Updated Schematic
Parts:
- removed BT1: 1042, Keystone-1042-*, symbol Digi:1042
- removed D3: BAT60JFILM, SOD2513X117N, symbol DiodeV2:BAT60JFILM
- removed IC1: DW01A-G, SOT95P280X135-6N, symbol BProtect:DW01A-G
- removed J5, J7: Header-Male-2.54_1x6, symbol Connector:Conn_01x06_Male
- removed J6: MICROXNJ, MICROXNJ, symbol MicroB:MICROXNJ
- removed J8: TP4056, SOIC127P600X175-9N, symbol TPBat:TP4056
- removed Q1: FS8205A, SOP65P640X120-8N, symbol MOS:FS8205A
- removed R1, R2, R3, R5: 1K, symbol Device:R_Small_US
- removed R4: 200, symbol Device:R_Small_US
- removed R6: 100, symbol Device:R_Small_US
- added D3: BAT60JFILM, BAT60:SOD2513X117N, symbol BAT60JFILM:BAT60JFILM
- added IC1: DW01A-G, DW:SOT95P280X135-6N, symbol DW01A-G:DW01A-G
- added J3: MICROXNJ, MICRO:MICROXNJ, symbol MICROXNJ:MICROXNJ
- added J4: TP4056, TP4056:SOIC127P600X175-9N, symbol TP4056:TP4056
- added J5: Conn_01x02_Male, Connector_PinHeader_2.54mm:PinHeader_1x02_P2.54mm_Vertical, symbol Connector:Conn_01x02_Male
- added J6: Conn_01x03_Male, Connector_PinHeader_2.54mm:PinHeader_1x03_P2.54mm_Vertical, symbol Connector:Conn_01x03_Male
- added Q1: FS8205A, FS82:SOP65P640X120-8N, symbol FS8205A:FS8205A
- added R1, R2, R3, R4: 1K, 1K_R:RESC1005X40N, symbol Device:R
- added R5: 100, 100_R:RESC1608X55N, symbol Device:R
- added TP1: GND, TestPoint:TestPoint_Pad_1.0x1.0mm, symbol Connector:TestPoint
- added TP2: 5V, TestPoint:TestPoint_Pad_1.0x1.0mm, symbol Connector:TestPoint
- added TP3: 3V3, TestPoint:TestPoint_Pad_1.0x1.0mm, symbol Connector:TestPoint
- added U2: 1024, BT:1024, symbol 1042:1024
- C1, C3, C4, C5: footprint (none) -> 10uFcapa:CAPC1608X100N
- C2: value CAP -> 10uF; footprint (none) -> 10uFcapa:CAPC1608X100N
- D1: value Green -> GREEN; footprint LED_THT:LED_D5.0mm_IRGrey -> LED_:LEDC1005X55N
- D2: value Red -> RED; footprint LED_THT:LED_D5.0mm_IRGrey -> LED_:LEDC1005X55N
- renumbered U3 to U1
Connections:
- net GND: now also J3.5, J4.1 (TEMP1), J4.3 (GND_3), J5.2 (Pin_2), J6.1 (Pin_1), Q1.2 (S1_1), Q1.3 (S1_2), R3.2, R4.1, TP1.1
- net OC: now also IC1.3 (OC), Q1.4 (G1)
- net OD: now also IC1.1 (OD), Q1.5 (G2)
- net V_out: now also D3.1, J6.2 (Pin_2), TP3.1
- net at D1.1 (K): now also R1.1
- net at D2.1 (K): now also R2.1
- net +5V renamed VCC
- net VCC: now also J3.1, J4.4 (VCC4), J4.8 (CE), J5.1 (Pin_1), TP2.1
- net BAT+ renamed VI
- net VI: now also J6.3 (Pin_3); no longer C2.2, C4.2
- net BAT-: no longer names the net of C4.1
- net BAT-: now also C2.2, J4.5 (BAT), R5.2, U2.1 (+)
- net V0: no longer names the net of C5.1, U1.2 (VO)
- net V0: now also D3.2
- new net: C4.2, IC1.6 (GND), Q1.6 (S2_1), Q1.7 (S2_2), U2.2 (-)
- new net: IC1.5 (VCC), R5.1
- new net: J4.2 (PROG2), R3.1
- new net: J4.6 (~{STDBY}), R1.2
- new net: J4.7 (~{CHRG}), R2.2
- new net: J3.MH1, J3.MH2, J3.MH3, J3.MH4, J3.MP1, J3.MP2
- new net: IC1.2 (CS), R4.2
- new net USB+: J3.3
- new net USB-: J3.2
Other:
- moved on the sheet: C4
