File: Design_Proposal/Power_SubModule/power.kicad_sch (KiCad schematic)
At the start: 23 parts, among them IC1 DW01A-G, J4 TP4056, J5 Conn_01x02_Male, J6 Conn_01x02_Male, Q1 FS8205A, U2 1024, U3 AMS1117-3.3

Commit message: Final Draft
Parts:
- removed J6: Conn_01x02_Male, Connector_PinHeader_2.54mm:PinHeader_1x02_P2.54mm_Vertical, symbol Connector:Conn_01x02_Male
- removed U3: AMS1117-3.3, Package_TO_SOT_SMD:SOT-223-3_TabPin2, symbol Regulator_Linear:AMS1117-3.3
- added J7, J9: Conn_01x02_Male, Connector_PinHeader_2.54mm:PinHeader_1x02_P2.54mm_Vertical, symbol Connector:Conn_01x02_Male
- added U1: HT75xx-1-SOT89, Package_TO_SOT_SMD:SOT-89-3, symbol Regulator_Linear:HT75xx-1-SOT89
- C1: renamed from C7; value 10u -> 10uF
- C2: renamed from C5; value 10u -> 10uF
- C3: renamed from C9; value 10u -> 10uF
- C5: renamed from C8; value 100n -> 10uF
- D1: value Green -> GREEN; footprint LED_THT:LED_D5.0mm_IRGrey -> LED_:LEDC1005X55N
- D2: value Red -> RED; footprint LED_THT:LED_D5.0mm_IRGrey -> LED_:LEDC1005X55N
- J6: renamed from J?; footprint (none) -> Connector_USB:USB_Micro-B_GCT_USB3076-30-A
- renumbered C2 to C4, J4 to J10, J5 to J8
Connections:
- net GND: now also U1.1 (GND); no longer J8.2 (Pin_2)
- net VI: now also C4.2, C5.1, J10.5 (BAT), R5.2, U2.1 (+), J7.1 (Pin_1); no longer C1.1
- net V_out: now also U1.3 (VOUT)
- net VCC: no longer names the net of C2.2, D1.2 (A), D2.2 (A), J10.4 (VCC4), J10.8 (CE)
- net VCC: now also J9.1 (Pin_1); no longer J6.1 (VBUS), J8.1 (Pin_1), TP2.1
- new net: C1.1, J7.2 (Pin_2), J8.1 (Pin_1), U1.2 (VIN)
- new net +5V: J6.1 (VBUS), J8.2 (Pin_2), J9.2 (Pin_2), TP2.1
Other:
- note removed: "Connectors"
- moved on the sheet: J8
