File: Design_Proposal/Main_Design/main.kicad_pcb (KiCad board)
At the start: 2 copper layers, 100.2 x 100.2 mm, 54 parts, among them IC1 DW01A-G, IC2 TMP102AIDRLR, J1 Conn_01x33_Female, J10 Conn_01x04_Male, J2 Conn_01x33_Female, J3 MICROXNJ, J4 TP4056, J5 Conn_01x02_Male, J6 Conn_01x02_Male, J7 Conn_01x03_Male, J8 Conn_01x05_Male, J9 Conn_01x06_Male, Q1 FS8205A, U1 AMS1117-3.3, U2 1024, U3 FT232RL-REEL, U4 M24C16-RMN6TP

Commit message: update pcb
Parts:
- added J2: Conn_01x33_Female, Connector_PinSocket_2.54mm:PinSocket_1x33_P2.54mm_Vertical, F.Cu at (168.0, 89.3)
- added J3: Conn_01x33_Female, Connector_PinSocket_2.54mm:PinSocket_1x33_P2.54mm_Vertical, F.Cu at (168.3, 149.7)
- added J4: Conn_01x10_Female, Connector_PinHeader_2.54mm:PinHeader_1x10_P2.54mm_Vertical, F.Cu at (101.2, 77.7)
- moved J11 59.3 mm to (111.8, 83.7), turned to -90 degrees
- moved J13 31.9 mm to (91.8, 76.0)
- moved C2 16.0 mm to (177.7, 77.0)
- moved R3 16.0 mm to (173.1, 76.7)
- moved D1 15.7 mm to (173.6, 62.4)
- moved R1 15.7 mm to (174.4, 64.6)
- moved D2 15.7 mm to (170.7, 64.8)
- moved R2 15.7 mm to (172.7, 64.6)
- moved C4 15.6 mm to (177.5, 68.3)
- moved J7 15.6 mm to (173.5, 70.7)
- moved C6 9.06 mm to (166.3, 127.1)
- moved TP4 9.06 mm to (163.6, 131.5)
- moved R6 9.06 mm to (163.9, 127.6)
- moved R7 9.06 mm to (158.3, 127.6)
- moved R8 9.06 mm to (160.5, 125.2)
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- renumbered C3 to C1, C1 to C2, C5 to C3, C2 to C4, C4 to C5, D4 to D3, D5 to D4, J7 to J10, J8 to J11, J9 to J12, J10 to J13, J2 to J5, J3 to J6, J4 to J7, J5 to J8, J6 to J9
Connections:
- net 3V3 renamed /microcontroller_interfacing/3V3
- C1 pad 1: /Power/VI -> /Power/V_IN
- C2 pad 2: VCC -> +5V
- C4 pad 2: Net-(C2-Pad2) -> /Power/V_IN
- C5 pad 1: Net-(C2-Pad2) -> /Power/V_IN
- C8 pad 1: VCC -> +5V
- C9 pad 1: VCC -> +5V
- D1 pad 2: VCC -> +5V
- D2 pad 2: VCC -> +5V
- J12 pad 1: VCC -> +5V
- J6 pad 1: VCC -> +5V
- J7 pad 4: VCC -> +5V
- J7 pad 5: Net-(C2-Pad2) -> /Power/V_IN
- J7 pad 8: VCC -> +5V
- J8 pad 1: VCC -> /Power/VCC
- J9 pad 2: /Power/VI -> /Power/V_IN
- R11 pad 1: VCC -> +5V
- R12 pad 1: VCC -> +5V
- R5 pad 2: Net-(C2-Pad2) -> /Power/V_IN
- TP2 pad 1: VCC -> +5V
- U1 pad 3: /Power/VI -> /Power/V_IN
- U2 pad 1: Net-(C2-Pad2) -> /Power/V_IN
- U3 pad 20: VCC -> +5V
- U3 pad 4: VCC -> +5V
- U4 pad 1: GND -> unconnected-(U4-Pad1)
- U4 pad 2: GND -> unconnected-(U4-Pad2)
- U4 pad 3: GND -> unconnected-(U4-Pad3)
Routing:
- net GND: track 102.1 -> 329.1 mm, vias 10 -> 11
- net VCC: track 136.0 -> 0.00 mm, vias 2 -> 0
- net +5V: track 0.00 -> 127.5 mm, vias 0 -> 2
- net V_out: track 273.0 -> 150.9 mm, vias 6 -> 4
- net Alert: track 76.2 -> 0.00 mm
- net Net-(C2-Pad2): track 63.5 -> 0.00 mm
- net /NRST: track 0.00 -> 60.4 mm, vias 0 -> 1
- net ADC1: track 56.3 -> 5.26 mm
- net /Power/V_IN: track 0.00 -> 38.0 mm
- net unconnected-(J7-Pad9): track 0.00 -> 27.5 mm
- net SCL2: track 22.1 -> 0.00 mm
- net /PC4: track 0.00 -> 22.1 mm
- net Write1: track 15.6 -> 0.00 mm
- net /PB0: track 0.00 -> 15.6 mm
- net /Power/VI: track 15.3 -> 0.00 mm
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
Commit message: Final PCB Design
Parts:
- removed J10: Conn_01x03_Male, Connector_PinHeader_2.54mm:PinHeader_1x03_P2.54mm_Vertical
- removed J11: Conn_01x05_Male, Connector_PinHeader_2.54mm:PinHeader_1x05_P2.54mm_Vertical
- removed J13: Conn_01x04_Male, Connector_PinHeader_2.54mm:PinHeader_1x04_P2.54mm_Vertical
- added J14: Conn_01x02_Male, Connector_PinHeader_2.54mm:PinHeader_1x02_P2.54mm_Vertical, F.Cu at (176.3, 112.1)
- added J15: Conn_01x02_Male, Connector_PinHeader_2.54mm:PinHeader_1x02_P2.54mm_Vertical, F.Cu at (174.4, 101.5)
- D3: value GREEN -> RED
- J12: value Conn_01x06_Male -> Conn_01x02_Male; footprint Connector_PinHeader_2.54mm:PinHeader_1x06_P2.54mm_Vertical -> Connector_PinHeader_2.54mm:PinHeader_1x02_P2.54mm_Vertical
- J6: value MICROXNJ -> USB_B_Micro; footprint MICRO:MICROXNJ -> Connector_USB:USB_Micro-B_GCT_USB3076-30-A
- U1: value AMS1117-3.3 -> HT7533-1; footprint Package_TO_SOT_SMD:SOT-223-3_TabPin2 -> Package_TO_SOT_SMD:SOT-89-3
- moved TP2 15.1 mm to (181.2, 99.8)
- moved C1 7.27 mm to (159.8, 74.1), turned to 0 degrees
- moved C3 6.64 mm to (160.7, 84.7), turned to 180 degrees
- moved J4 6.53 mm to (103.6, 83.8)
- moved J6 4.36 mm to (177.6, 121.5), turned to 90 degrees
- moved D4 4.19 mm to (167.0, 112.3)
- moved C10 4.11 mm to (90.4, 116.1)
- moved D3 3.81 mm to (166.6, 118.5)
- moved TP4 3.65 mm to (167.1, 132.4)
- moved R6 3.52 mm to (165.3, 124.4)
- moved R7 3.46 mm to (154.9, 127.0)
- moved TP5 3.32 mm to (154.9, 132.1)
- moved R4 3.03 mm to (138.7, 78.5), turned to 90 degrees
- moved R12 2.71 mm to (171.3, 112.2)
- moved TP3 2.68 mm to (171.2, 84.5)
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Connections:
- C1 pad 1: /Power/V_IN -> /Power/VI
- C10 pad 1: V_out -> +3V3
- C2 pad 2: +5V -> VCC
- C3 pad 1: V_out -> +3V3
- C4 pad 2: /Power/V_IN -> Net-(C4-Pad2)
- C5 pad 1: /Power/V_IN -> Net-(C4-Pad2)
- C6 pad 2: V_out -> +3V3
- C7 pad 1: /microcontroller_interfacing/3V3 -> 3V3_out
- C8 pad 1: +5V -> VCC
- C9 pad 1: +5V -> VCC
- D1 pad 2: +5V -> VCC
- D2 pad 2: +5V -> VCC
- IC2 pad 5: V_out -> +3V3
- J1 pad 1: V_out -> +3V3
- J12 pad 1: +5V -> USB+
- J12 pad 2: /microcontroller_interfacing/3V3 -> USB-
- J2 pad 1: V_out -> +3V3
- J6 pad 1: +5V -> Net-(J14-Pad1)
- J6 pad 4: unconnected-(J6-Pad4) -> GND
- J7 pad 4: +5V -> VCC
- J7 pad 5: /Power/V_IN -> Net-(C4-Pad2)
- J7 pad 8: +5V -> VCC
- J8 pad 1: /Power/VCC -> VCC
- J9 pad 1: V_out -> /Power/V_out
- J9 pad 2: /Power/V_IN -> /Power/VI
- R11 pad 1: +5V -> VCC
- R12 pad 1: +5V -> VCC
- R5 pad 2: /Power/V_IN -> Net-(C4-Pad2)
- R6 pad 1: V_out -> +3V3
- R7 pad 1: V_out -> +3V3
- R8 pad 1: V_out -> +3V3
- R9 pad 1: V_out -> +3V3
- TP2 pad 1: +5V -> VCC
- TP3 pad 1: V_out -> +3V3
- U1 pad 2: V_out -> /Power/VI
- U1 pad 3: /Power/V_IN -> +3V3
- U2 pad 1: /Power/V_IN -> Net-(C4-Pad2)
- U3 pad 17: /microcontroller_interfacing/3V3 -> 3V3_out
- U3 pad 20: +5V -> VCC
- U3 pad 4: +5V -> VCC
- U4 pad 1: unconnected-(U4-Pad1) -> GND
- U4 pad 2: unconnected-(U4-Pad2) -> GND
- U4 pad 3: unconnected-(U4-Pad3) -> GND
- U4 pad 8: V_out -> +3V3
Routing:
- net GND: track 329.1 -> 83.1 mm, vias 11 -> 5
- net +3V3: track 0.00 -> 228.0 mm, vias 0 -> 2
- net V_out: track 150.9 -> 0.00 mm, vias 4 -> 0
- net VCC: track 0.00 -> 109.6 mm, vias 0 -> 2
- net SDA1: track 71.1 -> 175.3 mm, vias 2 -> 3
- net SCL1: track 72.5 -> 167.9 mm
- net ADC1: track 5.26 -> 76.0 mm
- net Write1: track 0.00 -> 61.8 mm
- net SCL2: track 0.00 -> 56.0 mm, vias 0 -> 4
- net Net-(C4-Pad2): track 0.00 -> 52.8 mm, vias 0 -> 2
- net /NRST: track 60.4 -> 11.6 mm, vias 1 -> 0
- net /microcontroller_interfacing/3V3: track 48.6 -> 0.00 mm
- net SDA2: track 9.00 -> 54.6 mm
- net /Power/V_IN: track 38.0 -> 0.00 mm
- net 3V3_out: track 0.00 -> 37.7 mm, vias 0 -> 2
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