File: Design_Proposal/Main_Design/main.kicad_pcb (KiCad board)
At the start: 2 copper layers, 100.2 x 100.2 mm, 56 parts, among them IC1 DW01A-G, IC2 TMP102AIDRLR, J1 Conn_01x33_Female, J12 Conn_01x02_Male, J14 Conn_01x02_Male, J15 Conn_01x02_Male, J2 Conn_01x33_Female, J3 Conn_01x33_Female, J4 Conn_01x10_Female, J5 Conn_01x33_Female, J6 USB_B_Micro, J7 TP4056, J8 Conn_01x02_Male, J9 Conn_01x02_Male, Q1 FS8205A, U1 HT7533-1, U2 1024, U3 FT232RL-REEL, U4 M24C16-RMN6TP

Commit message: update
Parts:
- removed the C8 at (153.3, 121.0)
- removed C9: 100nF, 100NF_C:CAPC1005X55N
- removed D3, D4: RED, LED_:LEDC1005X55N
- removed J14, J15: Conn_01x02_Male, Connector_PinHeader_2.54mm:PinHeader_1x02_P2.54mm_Vertical
- removed R11, R12: 1K, 1K_R:RESC1005X40N
- added J10: Conn_01x03_Male, Connector_PinHeader_2.54mm:PinHeader_1x03_P2.54mm_Vertical, F.Cu at (218.9, 88.2)
- added J11: Conn_01x05_Male, Connector_PinHeader_2.54mm:PinHeader_1x05_P2.54mm_Vertical, F.Cu at (214.2, 88.2)
- IC2: value TMP102AIDRLR -> LM75AD,118; footprint TEMP_SENSOR:SOTFL50P160X60-6N -> LM75:SOIC127P600X175-8N
- J6: value USB_B_Micro -> MICROXNJ; footprint Connector_USB:USB_Micro-B_GCT_USB3076-30-A -> MICRO:MICROXNJ
- TP4: value SDA1 -> OS
- TP5: value Alert -> SCL1
- TP6: value SCL1 -> SDA1
- TP8: value RXD -> TXD
- TP9: value TXD -> RXD
- U1: value HT7533-1 -> AMS1117-3.3; footprint Package_TO_SOT_SMD:SOT-89-3 -> Package_TO_SOT_SMD:SOT-223-3_TabPin2
- U3: value FT232RL-REEL -> CH340C; footprint FT23:SOP65P780X200-28N -> CH340:SOIC127P600X180-16N
- moved TP9 68.4 mm to (200.9, 107.0)
- moved TP8 68.3 mm to (197.8, 107.0)
- moved C7 50.5 mm to (197.7, 109.5), turned to 0 degrees
- moved U3 49.6 mm to (192.3, 116.5)
- moved R7 45.8 mm to (200.6, 130.8), turned to 0 degrees
- moved TP5 45.5 mm to (200.2, 136.8)
- moved TP6 39.0 mm to (199.9, 133.8)
- moved J6 38.0 mm to (193.5, 86.9), turned to 0 degrees
- moved TP4 37.2 mm to (204.3, 130.8)
- moved U1 35.2 mm to (192.9, 98.1)
- moved C6 34.9 mm to (202.8, 133.3), turned to 0 degrees
- moved R8 34.7 mm to (192.0, 137.3), turned to 0 degrees
- moved R6 33.7 mm to (196.5, 137.3), turned to 0 degrees
- moved IC2 33.3 mm to (194.1, 132.6)
- renumbered C10 to C8
Connections:
- C1 pad 1: /Power/VI -> /Power/V_IN
- C2 pad 2: VCC -> +5V
- C3 pad 1: +3V3 -> V_out
- C4 pad 2: Net-(C4-Pad2) -> /Power/V_IN
- C5 pad 1: Net-(C4-Pad2) -> /Power/V_IN
- C6 pad 2: +3V3 -> V_out
- C7 pad 1: 3V3_out -> VCC
- D1 pad 2: VCC -> +5V
- D2 pad 2: VCC -> +5V
- IC2 pad 1: SCL1 -> SDA1
- IC2 pad 2: GND -> SCL1
- IC2 pad 3: Alert -> OS
- IC2 pad 5: +3V3 -> GND
- IC2 pad 6: SDA1 -> GND
- J3 pad 9: Alert -> OS
- J5 pad 9: Alert -> OS
- J6 pad 1: Net-(J14-Pad1) -> +5V
- J6 pad 4: GND -> unconnected-(J6-Pad4)
- J7 pad 4: VCC -> +5V
- J7 pad 5: Net-(C4-Pad2) -> /Power/V_IN
- J7 pad 8: VCC -> +5V
- J8 pad 1: VCC -> /Power/VCC
- J9 pad 1: /Power/V_out -> V_out
- J9 pad 2: /Power/VI -> /Power/V_IN
- R5 pad 2: Net-(C4-Pad2) -> /Power/V_IN
- R6 pad 1: +3V3 -> V_out
- R6 pad 2: SDA1 -> OS
- R7 pad 1: +3V3 -> V_out
- R7 pad 2: Alert -> SCL1
- R8 pad 1: +3V3 -> V_out
- R8 pad 2: SCL1 -> SDA1
- R9 pad 1: +3V3 -> V_out
- TP2 pad 1: VCC -> +5V
- TP3 pad 1: +3V3 -> V_out
- TP4 pad 1: SDA1 -> OS
- TP5 pad 1: Alert -> SCL1
- TP6 pad 1: SCL1 -> SDA1
- TP8 pad 1: RXD -> TXD
- TP9 pad 1: TXD -> RXD
- U1 pad 2: /Power/VI -> V_out
- U1 pad 3: +3V3 -> /Power/V_IN
- U2 pad 1: Net-(C4-Pad2) -> /Power/V_IN
- U3 pad 1: TXD -> GND
- U3 pad 15: USB+ -> unconnected-(U3-Pad15)
- U3 pad 16: USB- -> VCC
- U3 pad 2: unconnected-(U3-Pad2) -> TXD
- U3 pad 3: unconnected-(U3-Pad3) -> RXD
- U3 pad 5: RXD -> USB+
- U3 pad 6: unconnected-(U3-Pad6) -> USB-
- U3 pad 7: GND -> unconnected-(U3-Pad7)
- U3 pad 8: (no net) -> unconnected-(U3-Pad8)
Routing:
- net VCC: track 109.6 -> 0.00 mm, vias 2 -> 0
- net +5V: track 148.2 -> 257.8 mm, vias 2 -> 4
- net (no net): track 0.00 -> 103.9 mm, vias 0 -> 6
- net /Power/V_IN: track 0.00 -> 66.5 mm, vias 0 -> 2
- net Net-(C4-Pad2): track 52.8 -> 0.00 mm, vias 2 -> 0
- net 3V3_out: track 37.7 -> 0.00 mm, vias 2 -> 0
- net OS: track 0.00 -> 31.8 mm
- net Alert: track 31.8 -> 0.00 mm
- net Net-(D4-Pad1): track 22.9 -> 0.00 mm
- net Net-(D3-Pad1): track 20.7 -> 0.00 mm, vias 2 -> 0
- net /Power/VI: track 13.7 -> 0.00 mm
- net Net-(J14-Pad1): track 13.3 -> 0.00 mm, vias 2 -> 0
- net Net-(D3-Pad2): track 4.94 -> 0.00 mm
- net Net-(D4-Pad2): track 4.33 -> 0.00 mm

Commit message: update
Parts:
- removed the J10 at (218.9, 88.2)
- removed the J11 at (214.2, 88.2)
- added J7: Conn_01x02_Male, Connector_PinHeader_2.54mm:PinHeader_1x02_P2.54mm_Vertical, F.Cu at (181.1, 81.8)
- J6: value MICROXNJ -> USB_B_Micro; footprint MICRO:MICROXNJ -> Connector_USB:USB_Micro-B_GCT_USB3076-30-A
- U1: value AMS1117-3.3 -> HT75xx-1-SOT89; footprint Package_TO_SOT_SMD:SOT-223-3_TabPin2 -> Package_TO_SOT_SMD:SOT-89-3
- moved TP9 74.9 mm to (126.1, 111.0)
- moved TP8 68.3 mm to (129.6, 109.3)
- moved TP4 56.9 mm to (147.4, 132.9)
- moved R6 55.4 mm to (141.8, 128.6), turned to -90 degrees
- moved U3 52.8 mm to (139.6, 113.3)
- moved R7 51.8 mm to (150.4, 118.0), turned to 180 degrees
- moved C7 50.6 mm to (147.2, 108.8)
- moved TP5 49.6 mm to (150.8, 132.7)
- moved IC2 46.5 mm to (148.3, 124.7), turned to -90 degrees
- moved TP6 45.4 mm to (154.5, 132.7)
- moved J9 43.5 mm to (180.2, 105.1), turned to 0 degrees
- moved C6 43.2 mm to (160.1, 126.9), turned to 90 degrees
- moved R8 38.7 mm to (154.6, 127.2), turned to -90 degrees
- moved J6 38.1 mm to (177.4, 121.5), turned to 90 degrees
- moved U1 37.0 mm to (161.2, 79.0), turned to 90 degrees
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- renumbered J7 to J10, J12 to J11
Connections:
- C1 pad 1: /Power/V_IN -> Net-(C1-Pad1)
- C2 pad 2: +5V -> Net-(C2-Pad2)
- C4 pad 2: /Power/V_IN -> /Power/VI
- C5 pad 1: /Power/V_IN -> /Power/VI
- C7 pad 1: VCC -> V_out
- C8 pad 1: +3V3 -> V_out
- D1 pad 2: +5V -> Net-(C2-Pad2)
- D2 pad 2: +5V -> Net-(C2-Pad2)
- J1 pad 1: +3V3 -> V_out
- J10 pad 4: +5V -> Net-(C2-Pad2)
- J10 pad 5: /Power/V_IN -> /Power/VI
- J10 pad 8: +5V -> Net-(C2-Pad2)
- J2 pad 1: +3V3 -> V_out
- J6 pad 4: unconnected-(J6-Pad4) -> GND
- J8 pad 1: /Power/VCC -> Net-(C1-Pad1)
- J8 pad 2: GND -> +5V
- J9 pad 1: V_out -> Net-(C2-Pad2)
- J9 pad 2: /Power/V_IN -> +5V
- R5 pad 2: /Power/V_IN -> /Power/VI
- U1 pad 2: V_out -> Net-(C1-Pad1)
- U1 pad 3: /Power/V_IN -> V_out
- U2 pad 1: /Power/V_IN -> /Power/VI
- U3 pad 16: VCC -> V_out
- U3 pad 4: VCC -> V_out
- U4 pad 8: +3V3 -> V_out
Routing:
- net +3V3: track 228.0 -> 0.00 mm, vias 2 -> 0
- net V_out: track 0.00 -> 223.8 mm, vias 0 -> 4
- net (no net): track 103.9 -> 0.00 mm, vias 6 -> 0
- net +5V: track 257.8 -> 184.9 mm, vias 4 -> 5
- net /Power/V_IN: track 66.5 -> 0.00 mm, vias 2 -> 0
- net /Power/VI: track 0.00 -> 66.0 mm, vias 0 -> 2
- net Net-(C2-Pad2): track 0.00 -> 59.6 mm, vias 0 -> 4
- net USB+: track 72.4 -> 110.7 mm, vias 2 -> 4
- net Net-(C1-Pad1): track 0.00 -> 34.4 mm, vias 0 -> 4
- net GND: track 83.1 -> 50.6 mm, vias 5 -> 6
- net USB-: track 76.0 -> 105.0 mm
- net RXD: track 46.7 -> 38.9 mm
- net OS: track 31.8 -> 38.5 mm
- net TXD: track 45.0 -> 38.4 mm
- net SCL1: track 167.9 -> 164.7 mm
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Other:
- board size 100.2 x 100.2 mm -> 100 x 100 mm
