File: Design_Proposal/Main_Design/microcontroller_interfacing.kicad_sch (KiCad schematic)
At the start: 16 parts, among them J10 Conn_01x04_Male, J9 Conn_01x06_Male, U3 FT232RL-REEL, U4 M24C16-RMN6TP

Commit message: main project
Parts:
- renumbered D4 to D3, D5 to D4, J9 to J12, J10 to J13
Connections:
- net RXD: now also J12.4 (Pin_4); no longer J12.6 (Pin_6)
- net SDA2: now also J13.2 (Pin_2); no longer J13.4 (Pin_4)
- net TXD: now also J12.3 (Pin_3); no longer J12.5 (Pin_5)
- net USB+: now also J12.2 (Pin_2); no longer J12.3 (Pin_3)
- net USB-: now also J12.1 (Pin_1); no longer J12.4 (Pin_4)
- net VCC: now also J12.6 (Pin_6); no longer J12.1 (Pin_1)
- net V_out: now also J13.4 (Pin_4); no longer C10.1, J13.1 (Pin_1), U4.8 (VCC)
- net Write1: now also J13.1 (Pin_1); no longer J13.2 (Pin_2)
- net 3V3 renamed 3V3_out
- net 3V3_out: now also J12.5 (Pin_5); no longer J12.2 (Pin_2)
- new net +3V3: C10.1, U4.8 (VCC)
Other:
- note added: "(USB TO UART)"
- note added: "EEPROM"
- note added: "FTDI"
- note added: "LED's indicate FTDI is receiving(red) or transmitting data(green) Test points added for debugging purposes"
- note added: "Sub-circuit is used to convert USB to UART via the TXD and RXD pins of the FT232 C7,C8,C9 act as decoupling capacitors to filter out noise on the lines. All unused pins are not connected. Test points added for debugging purposes"
- note added: "This circuit consists of the EEPROM which will be used to store all the data collected by the sensing module. Pin7(WC) will connect directly to STM32 to proetct data from unplanned write operations Pins 1 to 3 are not used so grounded Pins 5 and 6 (SCL2 and SDA2) will connect directly to STM32 Test points added for debugging purposes"
- moved on the sheet: C7, C8, C9, D3, D4, J12, R11, R12, TP8, TP9, U3

Commit message: Final PCB Design
Parts:
- removed J12: Conn_01x06_Male, Connector_PinHeader_2.54mm:PinHeader_1x06_P2.54mm_Vertical, symbol Connector:Conn_01x06_Male
- removed J13: Conn_01x04_Male, Connector_PinHeader_2.54mm:PinHeader_1x04_P2.54mm_Vertical, symbol Connector:Conn_01x04_Male
- added J12: Conn_01x02_Male, Connector_PinHeader_2.54mm:PinHeader_1x02_P2.54mm_Vertical, symbol Connector:Conn_01x02_Male
- D3: value GREEN -> RED
Connections:
- net USB+: now also J12.1 (Pin_1)
- net USB-: now also J12.2 (Pin_2)
