File: Design_Proposal/Main_Design/main.kicad_sch (KiCad schematic)
At the start: 2 parts, among them J1 Conn_01x33_Female, J2 Conn_01x33_Female

Commit message: main schematic
Parts:
- added J2, J3: Conn_01x33_Female, Connector_PinSocket_2.54mm:PinSocket_1x33_P2.54mm_Vertical, symbol Connector:Conn_01x33_Female
- added J4: Conn_01x10_Female, Connector_PinHeader_2.54mm:PinHeader_1x10_P2.54mm_Vertical, symbol Connector:Conn_01x10_Female
- renumbered J2 to J5
Connections:
- net +5V: now also J3.1 (Pin_1), J4.1 (Pin_1)
- net ADC1: now also J2.11 (Pin_11), J4.2 (Pin_2)
- net Alert: now also J3.9 (Pin_9)
- net BOOT: now also J3.6 (Pin_6)
- net GND: now also J2.2 (Pin_2), J2.33 (Pin_33), J2.9 (Pin_9), J3.2 (Pin_2), J3.33 (Pin_33), J4.10 (Pin_10)
- net NRST: now also J2.10 (Pin_10)
- net PA0: now also J2.15 (Pin_15)
- net PA1: now also J2.16 (Pin_16)
- net PA10: now also J3.23 (Pin_23)
- net PA11: now also J3.22 (Pin_22)
- net PA12: now also J3.21 (Pin_21)
- net PA13: now also J3.20 (Pin_20)
- net PA14: now also J3.17 (Pin_17)
- net PA15: now also J3.16 (Pin_16)
- net PA4: now also J2.21 (Pin_21)
- net PA5: now also J2.22 (Pin_22)
- net PA6: now also J2.23 (Pin_23)
- net PA7: now also J2.24 (Pin_24)
- net PA8: now also J3.25 (Pin_25)
- net PA9: now also J3.24 (Pin_24)
- net PB0: now also J2.27 (Pin_27)
- net PB1: now also J2.28 (Pin_28)
- net PB13: now also J3.32 (Pin_32)
- net PB14: now also J3.31 (Pin_31)
- net PB15: now also J3.30 (Pin_30)
- net PB2: now also J2.29 (Pin_29)
- net PB3: now also J3.11 (Pin_11)
- net PB4: now also J3.10 (Pin_10)
- net PB8: now also J3.4 (Pin_4)
- net PB9: now also J3.3 (Pin_3)
- net PC1: now also J2.12 (Pin_12)
- net PC10: now also J3.15 (Pin_15)
- net PC11: now also J3.14 (Pin_14)
- net PC12: now also J3.13 (Pin_13)
- net PC13: now also J2.4 (Pin_4)
- net PC14: now also J2.5 (Pin_5)
- net PC15: now also J2.6 (Pin_6)
- net PC2: now also J2.13 (Pin_13)
- net PC3: now also J2.14 (Pin_14)
- net PC4: now also J2.25 (Pin_25)
- net PC5: now also J2.26 (Pin_26)
- net PC6: now also J3.29 (Pin_29)
- net PC7: now also J3.28 (Pin_28)
- net PC8: now also J3.27 (Pin_27)
- net PC9: now also J3.26 (Pin_26)
- net PD2: now also J3.12 (Pin_12)
- net PF0: now also J2.7 (Pin_7)
- net PF1: now also J2.8 (Pin_8)
- net PF4: now also J2.19 (Pin_19)
- net PF5: now also J2.20 (Pin_20)
- net PF6: now also J3.19 (Pin_19)
- net PF7: now also J3.18 (Pin_18)
- net RXD: now also J2.18 (Pin_18), J4.9 (Pin_9)
- net SCL1: now also J3.8 (Pin_8), J4.4 (Pin_4)
- net SCL2: now also J2.30 (Pin_30), J4.6 (Pin_6)
- net SDA1: now also J3.7 (Pin_7), J4.3 (Pin_3)
- net SDA2: now also J2.31 (Pin_31), J4.5 (Pin_5)
- net TXD: now also J2.17 (Pin_17), J4.8 (Pin_8)
- net VBAT: now also J2.3 (Pin_3)
- net VDD: now also J3.5 (Pin_5)
- net V_out: now also J2.1 (Pin_1)
- net Write1: now also J2.32 (Pin_32), J4.7 (Pin_7)
Other:
- note added: "Debug Connector"
- note removed: "Testpoints"
- moved on the sheet: J1, J5

Commit message: main project
Connections:
- net V_out renamed +3V3

Commit message: Final PCB Design
Changed lines of the file:
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@@
     )
   )
-  (sheet (at 28.575 29.21) (size 37.465 28.575) (fields_autoplaced)
+  (sheet (at 29.845 29.21) (size 37.465 28.575) (fields_autoplaced)
     (stroke (width 0.1524) (type solid) (color 0 0 0 0))
     (fill (color 0 0 0 0.0000))
-    (property "Sheet name" "Power" (id 0) (at 28.575 28.4984 0)
+    (property "Sheet name" "Power" (id 0) (at 29.845 28.4984 0)
       (effects (font (size 1.27 1.27)) (justify left bottom))
     )
-    (property "Sheet file" "power.kicad_sch" (id 1) (at 28.575 58.3696 0)
+    (property "Sheet file" "power.kicad_sch" (id 1) (at 29.845 58.3696 0)
       (effects (font (size 1.27 1.27)) (justify left top))
     )
@@
     )
     (path "/59b42903-2dc7-4011-ab5b-d7b81bd233c3/91b1f25b-dcb3-47ed-8828-3984e3f95572"
-      (reference "D3") (unit 1) (value "GREEN") (footprint "LED_:LEDC1005X55N")
+      (reference "D3") (unit 1) (value "RED") (footprint "LED_:LEDC1005X55N")
     )
     (path "/59b42903-2dc7-4011-ab5b-d7b81bd233c3/0607a974-1f7e-427f-9a87-182944959eab"
@@
     )
     (path "/d15c8919-7ccc-44b2-8fc4-b04c1b47b6fa/39125f99-6caa-4e69-9ae5-ca3bd6e3a49c"
-      (reference "J6") (unit 1) (value "USB_B_Micro") (footprint "")
+      (reference "J6") (unit 1) (value "USB_B_Micro") (footprint "Connector_USB:USB_Micro-B_GCT_USB3076-30-A")
     )
     (path "/d15c8919-7ccc-44b2-8fc4-b04c1b47b6fa/5b88f865-b1bf-4f4c-b514-21a095fc69fb"
@@
       (reference "J9") (unit 1) (value "Conn_01x02_Male") (footprint "Connector_PinHeader_2.54mm:PinHeader_1x02_P2.54mm_Vertical")
     )
-    (path "/cf6c12a4-3d95-473d-bafe-8be3892a84e9/d54417e2-94fc-493e-ad4d-f9d40ff34ff3"
-      (reference "J10") (unit 1) (value "Conn_01x03_Male") (footprint "Connector_PinHeader_2.54mm:PinHeader_1x03_P2.54mm_Vertical")
-    )
-    (path "/cf6c12a4-3d95-473d-bafe-8be3892a84e9/c4fc06e0-ba11-463d-a1e8-4c60d86fda87"
-      (reference "J11") (unit 1) (value "Conn_01x05_Male") (footprint "Connector_PinHeader_2.54mm:PinHeader_1x05_P2.54mm_Vertical")
-    )
-    (path "/59b42903-2dc7-4011-ab5b-d7b81bd233c3/8ff64f38-a2e3-4bbb-baed-409c7b708a82"
-      (reference "J12") (unit 1) (value "Conn_01x06_Male") (footprint "Connector_PinHeader_2.54mm:PinHeader_1x06_P2.54mm_Vertical")
-    )
-    (path "/59b42903-2dc7-4011-ab5b-d7b81bd233c3/a53e0776-e5b6-4c20-b49f-b16b81bee5b6"
-      (reference "J13") (unit 1) (value "Conn_01x04_Male") (footprint "Connector_PinHeader_2.54mm:PinHeader_1x04_P2.54mm_Vertical")
+    (path "/59b42903-2dc7-4011-ab5b-d7b81bd233c3/552e5b91-0f6d-4e5e-8efe-ed5a448c306b"
+      (reference "J12") (unit 1) (value "Conn_01x02_Male") (footprint "Connector_PinHeader_2.54mm:PinHeader_1x02_P2.54mm_Vertical")
+    )
+    (path "/d15c8919-7ccc-44b2-8fc4-b04c1b47b6fa/ec33585b-877f-4118-ae3a-7c6f1f5ecb59"
+      (reference "J14") (unit 1) (value "Conn_01x02_Male") (footprint "Connector_PinHeader_2.54mm:PinHeader_1x02_P2.54mm_Vertical")
+    )
+    (path "/d15c8919-7ccc-44b2-8fc4-b04c1b47b6fa/16974a66-63ee-4d75-91d2-5bffd655f5b6"
+      (reference "J15") (unit 1) (value "Conn_01x02_Male") (footprint "Connector_PinHeader_2.54mm:PinHeader_1x02_P2.54mm_Vertical")
     )
     (path "/d15c8919-7ccc-44b2-8fc4-b04c1b47b6fa/c61227ad-7e5c-47d6-b269-39d32e2c5b89"
@@
       (reference "TP11") (unit 1) (value "SDA2") (footprint "TestPoint:TestPoint_Pad_1.0x1.0mm")
     )
-    (path "/d15c8919-7ccc-44b2-8fc4-b04c1b47b6fa/d1a87309-7ed7-463d-82ac-113232561416"
-      (reference "U1") (unit 1) (value "AMS1117-3.3") (footprint "Package_TO_SOT_SMD:SOT-223-3_TabPin2")
+    (path "/d15c8919-7ccc-44b2-8fc4-b04c1b47b6fa/3cbaf087-00a9-44ba-9009-69de62b3bab5"
+      (reference "U1") (unit 1) (value "HT7533-1") (footprint "Package_TO_SOT_SMD:SOT-89-3")
     )
     (path "/d15c8919-7ccc-44b2-8fc4-b04c1b47b6fa/066b7f68-bd1d-420d-abbb-142d6be69cdb"

Commit message: update
Connections:
- net Alert renamed OS

Commit message: update
Connections:
- net +3V3 renamed V_out
