File: Design_Proposal/Main_Design/power.kicad_sch (KiCad schematic)
At the start: 23 parts, among them IC1 DW01A-G, J3 MICROXNJ, J4 TP4056, J5 Conn_01x02_Male, J6 Conn_01x02_Male, Q1 FS8205A, U1 AMS1117-3.3, U2 1024

Commit message: main project
Parts:
- removed J3: MICROXNJ, MICRO:MICROXNJ, symbol MICROXNJ:MICROXNJ
- added J6: USB_B_Micro, symbol Connector:USB_B_Micro
- renumbered C3 to C1, C1 to C2, C5 to C3, C2 to C4, C4 to C5, J4 to J7, J5 to J8, J6 to J9
Connections:
- net GND: now also J6.4 (ID), J6.5 (GND), J6.6 (Shield)
- net USB+: now also J6.3 (D+)
- net USB-: now also J6.2 (D-)
- net VCC: now also J6.1 (VBUS)
- net V_out: no longer C3.1, TP3.1, U1.2 (VO)
- new net +3V3: C3.1, TP3.1, U1.2 (VO)
- no-connect marks 5 -> 4
Other:
- note added: "Battery"
- note added: "Reverse protection"
- note added: "USB connector"
- note added: "UVLO"

Commit message: Final PCB Design
Parts:
- removed U1: AMS1117-3.3, Package_TO_SOT_SMD:SOT-223-3_TabPin2, symbol Regulator_Linear:AMS1117-3.3
- added J14, J15: Conn_01x02_Male, Connector_PinHeader_2.54mm:PinHeader_1x02_P2.54mm_Vertical, symbol Connector:Conn_01x02_Male
- added U1: HT7533-1, Package_TO_SOT_SMD:SOT-89-3, symbol Regulator_Linear:HT75xx-1-SOT89
- J6: footprint (none) -> Connector_USB:USB_Micro-B_GCT_USB3076-30-A
Connections:
- net +3V3: now also J15.2 (Pin_2), U1.3 (VOUT)
- net GND: now also U1.1 (GND)
- net VCC: now also J14.2 (Pin_2); no longer J6.1 (VBUS)
- net VI: now also U1.2 (VIN)
- new net: J14.1 (Pin_1), J6.1 (VBUS)
- new net 3V3_out: J15.1 (Pin_1)

Commit message: update
Parts:
- removed J14, J15: Conn_01x02_Male, Connector_PinHeader_2.54mm:PinHeader_1x02_P2.54mm_Vertical, symbol Connector:Conn_01x02_Male
- removed J6: USB_B_Micro, Connector_USB:USB_Micro-B_GCT_USB3076-30-A, symbol Connector:USB_B_Micro
- added J6: MICROXNJ, MICRO:MICROXNJ, symbol MICROXNJ:MICROXNJ
- U1: value HT7533-1 -> HT75xx-1-SOT89
Connections:
- net +3V3 is gone; now on net V_out: C3.1, TP3.1, U1.3 (VOUT)
- net VI is gone; now on net V_IN: C1.1, J9.2 (Pin_2), U1.2 (VIN)
- net GND: now also J6.5
- net USB+: now also J6.3
- net USB-: now also J6.2
- net VCC: no longer C2.2, D1.2 (A), D2.2 (A), J7.4 (VCC4), J7.8 (CE), TP2.1
- net V_IN: now reaches C4.2, C5.1, J7.5 (BAT), R5.2, U2.1 (+)
- new net: J6.MH1, J6.MH2, J6.MH3, J6.MH4, J6.MP1, J6.MP2
- new net +5V: C2.2, D1.2 (A), D2.2 (A), J6.1, J7.4 (VCC4), J7.8 (CE), TP2.1
- no-connect marks 4 -> 5
Other:
- note removed: "Battery"
- note removed: "Reverse protection"
- note removed: "USB connector"
- note removed: "UVLO"
- moved on the sheet: TP1

Commit message: update
Parts:
- removed J6: MICROXNJ, MICRO:MICROXNJ, symbol MICROXNJ:MICROXNJ
- added J6: USB_B_Micro, Connector_USB:USB_Micro-B_GCT_USB3076-30-A, symbol Connector:USB_B_Micro
- added J7, J9: Conn_01x02_Male, Connector_PinHeader_2.54mm:PinHeader_1x02_P2.54mm_Vertical, symbol Connector:Conn_01x02_Male
- renumbered J8 to J10, J9 to J11, J7 to J8
Connections:
- net +5V is gone; now on net VCC: C2.2, D1.2 (A), D2.2 (A), J8.4 (VCC4), J8.8 (CE), TP2.1
- net GND: now also J6.4 (ID), J6.5 (GND), J6.6 (Shield)
- net USB+: now also J6.3 (D+)
- net USB-: now also J6.2 (D-)
- net VCC: now also J7.2 (Pin_2)
- net V_out: no longer C3.1, TP3.1, U1.3 (VOUT)
- net V_IN: no longer names the net of C4.2, C5.1, J8.5 (BAT), R5.2, U2.1 (+)
- net V_IN: no longer C1.1, J11.2 (Pin_2), U1.2 (VIN)
- new net: J6.1 (VBUS), J7.1 (Pin_1)
- new net +3V3: C3.1, J9.2 (Pin_2), TP3.1, U1.3 (VOUT)
- new net 3V3_out: J9.1 (Pin_1)
- new net VI: C1.1, J11.2 (Pin_2), U1.2 (VIN)
- no-connect marks 5 -> 4
Other:
- note added: "Battery"
- note added: "Reverse protection"
- note added: "USB connector"
- note added: "UVLO"
- moved on the sheet: TP1

Commit message: update
Parts:
- removed J11: Conn_01x02_Male, Connector_PinHeader_2.54mm:PinHeader_1x02_P2.54mm_Vertical, symbol Connector:Conn_01x02_Male
- renumbered J8 to J10, J9 to J7, J10 to J8, J7 to J9
Connections:
- net 3V3_out is gone; now on net VI: J7.1 (Pin_1)
- net GND: no longer J8.2 (Pin_2)
- net VI: now also C4.2, C5.1, J10.5 (BAT), R5.2, U2.1 (+); no longer C1.1, U1.2 (VIN)
- net V_out: now also C3.1, TP3.1, U1.3 (VOUT)
- net at J9.1 (Pin_1): now also C2.2, D1.2 (A), D2.2 (A), J10.4 (VCC4), J10.8 (CE); no longer J6.1 (VBUS)
- removed net +3V3: C3.1, J7.2 (Pin_2), TP3.1, U1.3 (VOUT)
- removed net VCC: C2.2, D1.2 (A), D2.2 (A), J10.4 (VCC4), J10.8 (CE), J8.1 (Pin_1), J9.2 (Pin_2), TP2.1
- new net: C1.1, J7.2 (Pin_2), J8.1 (Pin_1), U1.2 (VIN)
- new net +5V: J6.1 (VBUS), J8.2 (Pin_2), J9.2 (Pin_2), TP2.1
Other:
- note removed: "Connectors"
- moved on the sheet: J7, J8, J9
