File: Design_Proposal/Main_Design/sensing.kicad_sch (KiCad schematic)
At the start: 13 parts, among them IC2 TMP102AIDRLR, J7 Conn_01x03_Male, J8 Conn_01x05_Male

Commit message: main project
Parts:
- renumbered J7 to J10, J8 to J11
Connections:
- net V_out renamed +3V3
- net +3V3: no longer J10.3 (Pin_3), J11.5 (Pin_5)
- new net 3V3: J10.3 (Pin_3), J11.5 (Pin_5)
Changed lines of the file:
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@@
   (junction (at 41.91 125.095) (diameter 0) (color 0 0 0 0)
   )
+  (junction (at 55.88 40.005) (diameter 0) (color 0 0 0 0)
+  )
   (junction (at 51.435 125.095) (diameter 0) (color 0 0 0 0)
   )
@@
     (stroke (width 0) (type default) (color 0 0 0 0))
   )
+  (wire (pts (xy 55.88 40.005) (xy 55.88 45.72))
+    (stroke (width 0) (type default) (color 0 0 0 0))
+  )
   (wire (pts (xy 175.26 43.18) (xy 181.61 43.18))
     (stroke (width 0) (type default) (color 0 0 0 0))
@@
     (stroke (width 0) (type default) (color 0 0 0 0))
   )
+  (wire (pts (xy 93.345 111.125) (xy 93.345 118.745))
+    (stroke (width 0) (type default) (color 0 0 0 0))
+  )
+  (wire (pts (xy 91.44 145.415) (xy 93.345 145.415))
+    (stroke (width 0) (type default) (color 0 0 0 0))
+  )
+  (wire (pts (xy 91.44 142.875) (xy 93.345 142.875))
+    (stroke (width 0) (type default) (color 0 0 0 0))
+  )
+  (wire (pts (xy 55.88 36.83) (xy 55.88 40.005))
+    (stroke (width 0) (type default) (color 0 0 0 0))
+  )
+  (wire (pts (xy 64.77 54.61) (xy 71.12 54.61))
+    (stroke (width 0) (type default) (color 0 0 0 0))
+  )
+  (wire (pts (xy 41.91 145.415) (xy 43.815 145.415))
+    (stroke (width 0) (type default) (color 0 0 0 0))
+  )
   (wire (pts (xy 93.345 125.095) (xy 93.345 142.875))
     (stroke (width 0) (type default) (color 0 0 0 0))
   )
-  (wire (pts (xy 78.105 118.745) (xy 67.945 118.745))
-    (stroke (width 0) (type default) (color 0 0 0 0))
-  )
-  (wire (pts (xy 91.44 145.415) (xy 93.345 145.415))
-    (stroke (width 0) (type default) (color 0 0 0 0))
-  )
-  (wire (pts (xy 91.44 142.875) (xy 93.345 142.875))
-    (stroke (width 0) (type default) (color 0 0 0 0))
-  )
-  (wire (pts (xy 55.88 36.83) (xy 55.88 45.72))
-    (stroke (width 0) (type default) (color 0 0 0 0))
-  )
-  (wire (pts (xy 64.77 54.61) (xy 71.12 54.61))
-    (stroke (width 0) (type default) (color 0 0 0 0))
-  )
-  (wire (pts (xy 41.91 145.415) (xy 43.815 145.415))
-    (stroke (width 0) (type default) (color 0 0 0 0))
-  )
   (wire (pts (xy 41.91 125.095) (xy 33.02 125.095))
     (stroke (width 0) (type default) (color 0 0 0 0))
@@
     (stroke (width 0) (type default) (color 0 0 0 0))
   )
-  (wire (pts (xy 93.345 111.125) (xy 93.345 118.745))
-    (stroke (width 0) (type default) (color 0 0 0 0))
-  )
   (wire (pts (xy 93.345 149.86) (xy 36.83 149.86))
+    (stroke (width 0) (type default) (color 0 0 0 0))
+  )
+  (wire (pts (xy 67.945 118.745) (xy 78.105 118.745))
     (stroke (width 0) (type default) (color 0 0 0 0))
   )
@@
     (effects (font (size 2 2) bold) (justify left bottom))
   )
+  (global_label "3V3" (shape input) (at 175.26 38.1 180) (fields_autoplaced)
+    (effects (font (size 1.27 1.27)) (justify right))
+    (property "Intersheet References" "${INTERSHEET_REFS}" (id 0) (at 169.3393 38.1794 0)
+      (effects (font (size 1.27 1.27)) (justify right) hide)
+    )
+  )
   (global_label "Alert" (shape input) (at 40.64 139.065 180) (fields_autoplaced)
     (effects (font (size 1.27 1.27)) (justify right))
@@
     )
   )
-  (global_label "V_out" (shape input) (at 55.88 36.83 90) (fields_autoplaced)
-    (effects (font (size 1.27 1.27)) (justify left))
-    (property "Intersheet References" "${INTERSHEET_REFS}" (id 0) (at 55.8006 29.3369 90)
-      (effects (font (size 1.27 1.27)) (justify left) hide)
-    )
-  )
   (global_label "ADC1" (shape input) (at 167.64 40.64 180) (fields_autoplaced)
     (effects (font (size 1.27 1.27)) (justify right))
@@
     )
   )
-  (global_label "V_out" (shape input) (at 236.22 31.75 180) (fields_autoplaced)
-    (effects (font (size 1.27 1.27)) (justify right))
-    (property "Intersheet References" "${INTERSHEET_REFS}" (id 0) (at 228.7269 31.6706 0)
-      (effects (font (size 1.27 1.27)) (justify right) hide)
-    )
-  )
   (global_label "SCL1" (shape input) (at 50.165 134.62 180) (fields_autoplaced)
     (effects (font (size 1.27 1.27)) (justify right))
@@
     (property "Intersheet References" "${INTERSHEET_REFS}" (id 0) (at 221.8326 39.4494 0)
       (effects (font (size 1.27 1.27)) (justify right) hide)
-    )
-  )
-  (global_label "V_out" (shape input) (at 93.345 111.125 90) (fields_autoplaced)
-    (effects (font (size 1.27 1.27)) (justify left))
-    (property "Intersheet References" "${INTERSHEET_REFS}" (id 0) (at 93.2656 103.6319 90)
-      (effects (font (size 1.27 1.27)) (justify left) hide)
     )
   )
@@
     )
   )
-  (global_label "V_out" (shape input) (at 175.26 38.1 180) (fields_autoplaced)
-    (effects (font (size 1.27 1.27)) (justify right))
-    (property "Intersheet References" "${INTERSHEET_REFS}" (id 0) (at 167.7669 38.0206 0)
+  (global_label "3V3" (shape input) (at 236.22 31.75 180) (fields_autoplaced)
+    (effects (font (size 1.27 1.27)) (justify right))
+    (property "Intersheet References" "${INTERSHEET_REFS}" (id 0) (at 230.2993 31.8294 0)
       (effects (font (size 1.27 1.27)) (justify right) hide)
     )
@@
   (symbol (lib_id "power:GND") (at 51.435 162.56 0) (unit 1)
     (in_bom yes) (on_board yes) (fields_autoplaced)
-    (property "Reference" "#PWR012" (id 0) (at 51.435 168.91 0)
+    (property "Reference" "#PWR021" (id 0) (at 51.435 168.91 0)
       (effects (font (size 1.27 1.27)) hide)
     )
@@
   (symbol (lib_id "power:PWR_FLAG") (at 54.61 156.21 270) (unit 1)
     (in_bom yes) (on_board yes) (fields_autoplaced)
-    (property "Reference" "#FLG04" (id 0) (at 56.515 156.21 0)
+    (property "Reference" "#FLG03" (id 0) (at 56.515 156.21 0)
       (effects (font (size 1.27 1.27)) hide)
     )
@@
   (symbol (lib_id "power:GND") (at 106.68 146.685 0) (unit 1)
     (in_bom yes) (on_board yes) (fields_autoplaced)
-    (property "Reference" "#PWR015" (id 0) (at 106.68 153.035 0)
+    (property "Reference" "#PWR024" (id 0) (at 106.68 153.035 0)
       (effects (font (size 1.27 1.27)) hide)
     )
@@
     (pin "1")
   )
+  (symbol (lib_id "power:+3V3") (at 93.345 111.125 0) (unit 1)
+    (in_bom yes) (on_board yes) (fields_autoplaced)
+    (property "Reference" "#PWR0101" (id 0) (at 93.345 114.935 0)
+      (effects (font (size 1.27 1.27)) hide)
+    )
+    (property "Value" "+3V3" (id 1) (at 93.345 105.41 0))
+    (property "Footprint" "" (id 2) (at 93.345 111.125 0)
+      (effects (font (size 1.27 1.27)) hide)
+    )
+    (property "Datasheet" "" (id 3) (at 93.345 111.125 0)
+      (effects (font (size 1.27 1.27)) hide)
+    )
+    (pin "1")
+  )
+  (symbol (lib_id "power:PWR_FLAG") (at 55.88 40.005 270) (unit 1)
+    (in_bom yes) (on_board yes) (fields_autoplaced)
+    (property "Reference" "#FLG0103" (id 0) (at 57.785 40.005 0)
+      (effects (font (size 1.27 1.27)) hide)
+    )
+    (property "Value" "PWR_FLAG" (id 1) (at 59.69 40.0049 90)
+      (effects (font (size 1.27 1.27)) (justify left))
+    )
+    (property "Footprint" "" (id 2) (at 55.88 40.005 0)
+      (effects (font (size 1.27 1.27)) hide)
+    )
+    (property "Datasheet" "~" (id 3) (at 55.88 40.005 0)
+      (effects (font (size 1.27 1.27)) hide)
+    )
+    (pin "1")
+  )
   (symbol (lib_id "Device:R") (at 41.91 128.905 0) (unit 1)
     (in_bom yes) (on_board yes) (fields_autoplaced)
@@
   (symbol (lib_id "Connector:Conn_01x05_Male") (at 246.38 36.83 180) (unit 1)
     (in_bom yes) (on_board yes) (fields_autoplaced)
-    (property "Reference" "J8" (id 0) (at 247.65 35.5599 0)
+    (property "Reference" "J11" (id 0) (at 247.65 35.5599 0)
       (effects (font (size 1.27 1.27)) (justify right))
     )
@@
   (symbol (lib_id "power:GND") (at 55.88 71.12 0) (unit 1)
     (in_bom yes) (on_board yes) (fields_autoplaced)
-    (property "Reference" "#PWR013" (id 0) (at 55.88 77.47 0)
+    (property "Reference" "#PWR022" (id 0) (at 55.88 77.47 0)
       (effects (font (size 1.27 1.27)) hide)
     )
@@
   (symbol (lib_id "Connector:Conn_01x03_Male") (at 186.69 40.64 180) (unit 1)
     (in_bom yes) (on_board yes) (fields_autoplaced)
-    (property "Reference" "J7" (id 0) (at 187.96 39.3699 0)
+    (property "Reference" "J10" (id 0) (at 187.96 39.3699 0)
       (effects (font (size 1.27 1.27)) (justify right))
     )
@@
   (symbol (lib_id "power:GND") (at 67.945 118.745 270) (unit 1)
     (in_bom yes) (on_board yes) (fields_autoplaced)
-    (property "Reference" "#PWR014" (id 0) (at 61.595 118.745 0)
+    (property "Reference" "#PWR023" (id 0) (at 61.595 118.745 0)
       (effects (font (size 1.27 1.27)) hide)
     )
@@
       (effects (font (size 1.27 1.27)) hide)
     )
+    (pin "1")
+  )
+  (symbol (lib_id "power:+3V3") (at 55.88 36.83 0) (unit 1)
+    (in_bom yes) (on_board yes) (fields_autoplaced)
+    (property "Reference" "#PWR0105" (id 0) (at 55.88 40.64 0)
+      (effects (font (size 1.27 1.27)) hide)
+    )
+    (property "Value" "+3V3" (id 1) (at 55.88 31.75 0))
+    (property "Footprint" "" (id 2) (at 55.88 36.83 0)
+      (effects (font (size 1.27 1.27)) hide)
+    )
+    (property "Datasheet" "" (id 3) (at 55.88 36.83 0)
+      (effects (font (size 1.27 1.27)) hide)
+    )

Commit message: Final PCB Design
Parts:
- removed J10: Conn_01x03_Male, Connector_PinHeader_2.54mm:PinHeader_1x03_P2.54mm_Vertical, symbol Connector:Conn_01x03_Male
- removed J11: Conn_01x05_Male, Connector_PinHeader_2.54mm:PinHeader_1x05_P2.54mm_Vertical, symbol Connector:Conn_01x05_Male
Other:
- note removed: "ADC SENSOR CONNECTORS"
- note removed: "Connectors/Pin Headers"
- note removed: "DIGITAL SENSOR CONNECTORS"
Changed lines of the file:
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@@
     (stroke (width 0) (type default) (color 0 0 0 0))
   )
-  (wire (pts (xy 236.22 31.75) (xy 241.3 31.75))
-    (stroke (width 0) (type default) (color 0 0 0 0))
-  )
-  (wire (pts (xy 166.37 44.45) (xy 175.26 44.45))
-    (stroke (width 0) (type default) (color 0 0 0 0))
-  )
-  (polyline (pts (xy 140.97 76.2) (xy 284.48 76.2))
+  (polyline (pts (xy 12.7 85.09) (xy 284.48 85.09))
     (stroke (width 0) (type default) (color 0 0 0 0))
   )
@@
     (stroke (width 0) (type default) (color 0 0 0 0))
   )
-  (wire (pts (xy 175.26 43.18) (xy 181.61 43.18))
-    (stroke (width 0) (type default) (color 0 0 0 0))
-  )
   (wire (pts (xy 93.345 118.745) (xy 93.345 125.095))
     (stroke (width 0) (type default) (color 0 0 0 0))
   )
-  (wire (pts (xy 228.6 34.29) (xy 241.3 34.29))
-    (stroke (width 0) (type default) (color 0 0 0 0))
-  )
   (wire (pts (xy 50.165 134.62) (xy 51.435 134.62))
     (stroke (width 0) (type default) (color 0 0 0 0))
@@
     (stroke (width 0) (type default) (color 0 0 0 0))
   )
-  (wire (pts (xy 234.95 41.91) (xy 241.3 41.91))
-    (stroke (width 0) (type default) (color 0 0 0 0))
-  )
   (wire (pts (xy 33.02 149.86) (xy 33.02 132.715))
     (stroke (width 0) (type default) (color 0 0 0 0))
@@
     (stroke (width 0) (type default) (color 0 0 0 0))
   )
-  (wire (pts (xy 167.64 40.64) (xy 181.61 40.64))
-    (stroke (width 0) (type default) (color 0 0 0 0))
-  )
   (wire (pts (xy 55.88 66.04) (xy 55.88 71.12))
     (stroke (width 0) (type default) (color 0 0 0 0))
   )
-  (wire (pts (xy 175.26 38.1) (xy 181.61 38.1))
-    (stroke (width 0) (type default) (color 0 0 0 0))
-  )
   (wire (pts (xy 41.91 139.065) (xy 41.91 145.415))
     (stroke (width 0) (type default) (color 0 0 0 0))
@@
     (stroke (width 0) (type default) (color 0 0 0 0))
   )
-  (wire (pts (xy 228.6 39.37) (xy 241.3 39.37))
-    (stroke (width 0) (type default) (color 0 0 0 0))
-  )
-  (polyline (pts (xy 140.97 88.9) (xy 140.97 198.12))
-    (stroke (width 0) (type default) (color 0 0 0 0))
-  )
   (wire (pts (xy 43.815 145.415) (xy 60.96 145.415))
     (stroke (width 0) (type default) (color 0 0 0 0))
@@
     (stroke (width 0) (type default) (color 0 0 0 0))
   )
-  (polyline (pts (xy 12.7 88.9) (xy 140.97 88.9))
-    (stroke (width 0) (type default) (color 0 0 0 0))
-  )
   (wire (pts (xy 51.435 140.335) (xy 53.34 140.335))
     (stroke (width 0) (type default) (color 0 0 0 0))
   )
-  (polyline (pts (xy 140.97 12.7) (xy 140.97 88.9))
-    (stroke (width 0) (type default) (color 0 0 0 0))
-  )
   (wire (pts (xy 55.88 54.61) (xy 55.88 58.42))
     (stroke (width 0) (type default) (color 0 0 0 0))
   )
-  (wire (pts (xy 175.26 44.45) (xy 175.26 43.18))
-    (stroke (width 0) (type default) (color 0 0 0 0))
-  )
   (wire (pts (xy 93.345 149.86) (xy 93.345 145.415))
-    (stroke (width 0) (type default) (color 0 0 0 0))
-  )
-  (wire (pts (xy 220.98 36.83) (xy 241.3 36.83))
     (stroke (width 0) (type default) (color 0 0 0 0))
   )
@@
     (effects (font (size 1.27 1.27)) (justify left bottom))
   )
-  (text "Connectors/Pin Headers" (at 149.86 24.13 0)
-    (effects (font (size 2 2) bold) (justify left bottom))
-  )
-  (text "ADC SENSOR CONNECTORS\n" (at 173.355 48.895 0)
-    (effects (font (size 1.27 1.27)) (justify left bottom))
-  )
-  (text "DIGITAL SENSOR CONNECTORS\n" (at 234.95 46.99 0)
-    (effects (font (size 1.27 1.27)) (justify left bottom))
-  )
   (text "Analog Sensor\n" (at 16.51 25.4 0)
     (effects (font (size 2 2) bold) (justify left bottom))
-  )
-  (global_label "3V3" (shape input) (at 175.26 38.1 180) (fields_autoplaced)
-    (effects (font (size 1.27 1.27)) (justify right))
-    (property "Intersheet References" "${INTERSHEET_REFS}" (id 0) (at 169.3393 38.1794 0)
-      (effects (font (size 1.27 1.27)) (justify right) hide)
-    )
   )
   (global_label "Alert" (shape input) (at 40.64 139.065 180) (fields_autoplaced)
@@
     )
   )
-  (global_label "ADC1" (shape input) (at 167.64 40.64 180) (fields_autoplaced)
-    (effects (font (size 1.27 1.27)) (justify right))
-    (property "Intersheet References" "${INTERSHEET_REFS}" (id 0) (at 160.3888 40.7194 0)
-      (effects (font (size 1.27 1.27)) (justify right) hide)
-    )
-  )
   (global_label "SDA1" (shape input) (at 28.575 149.86 180) (fields_autoplaced)
     (effects (font (size 1.27 1.27)) (justify right))
@@
     )
   )
-  (global_label "Alert" (shape input) (at 228.6 39.37 180) (fields_autoplaced)
-    (effects (font (size 1.27 1.27)) (justify right))
-    (property "Intersheet References" "${INTERSHEET_REFS}" (id 0) (at 221.8326 39.4494 0)
-      (effects (font (size 1.27 1.27)) (justify right) hide)
-    )
-  )
   (global_label "ADC1" (shape input) (at 71.12 54.61 0) (fields_autoplaced)
     (effects (font (size 1.27 1.27)) (justify left))
     (property "Intersheet References" "${INTERSHEET_REFS}" (id 0) (at 78.3712 54.5306 0)
       (effects (font (size 1.27 1.27)) (justify left) hide)
-    )
-  )
-  (global_label "3V3" (shape input) (at 236.22 31.75 180) (fields_autoplaced)
-    (effects (font (size 1.27 1.27)) (justify right))
-    (property "Intersheet References" "${INTERSHEET_REFS}" (id 0) (at 230.2993 31.8294 0)
-      (effects (font (size 1.27 1.27)) (justify right) hide)
-    )
-  )
-  (global_label "GND" (shape input) (at 234.95 41.91 180) (fields_autoplaced)
-    (effects (font (size 1.27 1.27)) (justify right))
-    (property "Intersheet References" "${INTERSHEET_REFS}" (id 0) (at 228.6664 41.9894 0)
-      (effects (font (size 1.27 1.27)) (justify right) hide)
-    )
-  )
-  (global_label "SDA1" (shape input) (at 228.6 34.29 180) (fields_autoplaced)
-    (effects (font (size 1.27 1.27)) (justify right))
-    (property "Intersheet References" "${INTERSHEET_REFS}" (id 0) (at 221.4093 34.3694 0)
-      (effects (font (size 1.27 1.27)) (justify right) hide)
-    )
-  )
-  (global_label "SCL1" (shape input) (at 220.98 36.83 180) (fields_autoplaced)
-    (effects (font (size 1.27 1.27)) (justify right))
-    (property "Intersheet References" "${INTERSHEET_REFS}" (id 0) (at 213.8498 36.9094 0)
-      (effects (font (size 1.27 1.27)) (justify right) hide)
-    )
-  )
-  (global_label "GND" (shape input) (at 166.37 44.45 180) (fields_autoplaced)
-    (effects (font (size 1.27 1.27)) (justify right))
-    (property "Intersheet References" "${INTERSHEET_REFS}" (id 0) (at 160.0864 44.3706 0)
-      (effects (font (size 1.27 1.27)) (justify right) hide)
     )
   )
@@
     (pin "2")
   )
-  (symbol (lib_id "Connector:Conn_01x05_Male") (at 246.38 36.83 180) (unit 1)
-    (in_bom yes) (on_board yes) (fields_autoplaced)
-    (property "Reference" "J11" (id 0) (at 247.65 35.5599 0)
-      (effects (font (size 1.27 1.27)) (justify right))
-    )
-    (property "Value" "Conn_01x05_Male" (id 1) (at 247.65 38.0999 0)
-      (effects (font (size 1.27 1.27)) (justify right))
-    )
-    (property "Footprint" "Connector_PinHeader_2.54mm:PinHeader_1x05_P2.54mm_Vertical" (id 2) (at 246.38 36.83 0)
-      (effects (font (size 1.27 1.27)) hide)
-    )
-    (property "Datasheet" "~" (id 3) (at 246.38 36.83 0)
-      (effects (font (size 1.27 1.27)) hide)
-    )
-    (pin "1")
-    (pin "2")
-    (pin "3")
-    (pin "4")
-    (pin "5")
-  )
   (symbol (lib_id "power:GND") (at 55.88 71.12 0) (unit 1)
     (in_bom yes) (on_board yes) (fields_autoplaced)
@@
     (pin "1")
   )
-  (symbol (lib_id "Connector:Conn_01x03_Male") (at 186.69 40.64 180) (unit 1)
-    (in_bom yes) (on_board yes) (fields_autoplaced)
-    (property "Reference" "J10" (id 0) (at 187.96 39.3699 0)
-      (effects (font (size 1.27 1.27)) (justify right))
-    )
-    (property "Value" "Conn_01x03_Male" (id 1) (at 187.96 41.9099 0)
-      (effects (font (size 1.27 1.27)) (justify right))
-    )
-    (property "Footprint" "Connector_PinHeader_2.54mm:PinHeader_1x03_P2.54mm_Vertical" (id 2) (at 186.69 40.64 0)
-      (effects (font (size 1.27 1.27)) hide)
-    )
-    (property "Datasheet" "~" (id 3) (at 186.69 40.64 0)
-      (effects (font (size 1.27 1.27)) hide)
-    )
-    (pin "1")
-    (pin "2")
-    (pin "3")
-  )
   (symbol (lib_id "Device:R") (at 55.88 49.53 0) (unit 1)

Commit message: update
Parts:
- removed IC2: TMP102AIDRLR, TEMP_SENSOR:SOTFL50P160X60-6N, symbol TEMP:TMP102AIDRLR
- added IC2: LM75AD,118, SOIC127P600X175-8N, symbol LM75:LM75AD,118
- added J10: Conn_01x03_Male, Connector_PinHeader_2.54mm:PinHeader_1x03_P2.54mm_Vertical, symbol Connector:Conn_01x03_Male
- added J11: Conn_01x05_Male, Connector_PinHeader_2.54mm:PinHeader_1x05_P2.54mm_Vertical, symbol Connector:Conn_01x05_Male
- TP4: value SDA1 -> OS
- TP5: value Alert -> SCL1
- TP6: value SCL1 -> SDA1
Connections:
- net ADC1: now also J10.2 (Pin_2)
- net Alert: now also J11.2 (Pin_2); no longer R7.2, TP5.1
- net GND: now also IC2.4 (GND), IC2.5 (A2), IC2.6 (A1), IC2.7 (A0), J10.1 (Pin_1), J11.1 (Pin_1)
- net SCL1: now also R7.2, TP5.1, IC2.2 (SCL), J11.3 (Pin_3); no longer R8.2, TP6.1
- net SDA1: now also R8.2, TP6.1, IC2.1 (SDA), J11.4 (Pin_4); no longer R6.2, TP4.1
- net +3V3 renamed V_out
- net V_out: now also IC2.8 (VCC), J10.3 (Pin_3), J11.5 (Pin_5)
- new net OS: IC2.3 (OS), R6.2, TP4.1
Other:
- note added: "ADC SENSOR CONNECTORS"
- note added: "Connectors/Pin Headers"
- note added: "DIGITAL SENSOR CONNECTORS"

Commit message: update
Parts:
- IC2: footprint SOIC127P600X175-8N -> LM75:SOIC127P600X175-8N
Changed lines of the file:
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@@
     (property "Reference" "IC2" (id 0) (at 68.58 128.905 0))
     (property "Value" "LM75AD,118" (id 1) (at 68.58 131.445 0))
-    (property "Footprint" "SOIC127P600X175-8N" (id 2) (at 77.47 134.62 0)
+    (property "Footprint" "LM75:SOIC127P600X175-8N" (id 2) (at 77.47 134.62 0)
       (effects (font (size 1.27 1.27)) (justify left) hide)
     )

Commit message: update
Parts:
- renumbered J10 to J12, J11 to J13
Changed lines of the file:
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@@
   (symbol (lib_id "Connector:Conn_01x05_Male") (at 246.38 36.83 180) (unit 1)
     (in_bom yes) (on_board yes) (fields_autoplaced)
-    (property "Reference" "J11" (id 0) (at 247.65 35.5599 0)
+    (property "Reference" "J13" (id 0) (at 247.65 35.5599 0)
       (effects (font (size 1.27 1.27)) (justify right))
     )
@@
   (symbol (lib_id "Connector:Conn_01x03_Male") (at 186.69 40.64 180) (unit 1)
     (in_bom yes) (on_board yes) (fields_autoplaced)
-    (property "Reference" "J10" (id 0) (at 187.96 39.3699 0)
+    (property "Reference" "J12" (id 0) (at 187.96 39.3699 0)
       (effects (font (size 1.27 1.27)) (justify right))
     )
