File: Design_Proposal/Sensing_SubModule/sensing.kicad_sch (KiCad schematic)
At the start: 13 parts, among them IC2 TMP102AIDRLR, J7 Conn_01x03_Male, J8 Conn_01x05_Male

Commit message: Final Draft
Parts:
- removed IC2: TMP102AIDRLR, TEMP_SENSOR:SOTFL50P160X60-6N, symbol TEMP:TMP102AIDRLR
- removed J7: Conn_01x03_Male, Connector_PinHeader_2.54mm:PinHeader_1x03_P2.54mm_Vertical, symbol Connector:Conn_01x03_Male
- removed J8: Conn_01x05_Male, Connector_PinHeader_2.54mm:PinHeader_1x05_P2.54mm_Vertical, symbol Connector:Conn_01x05_Male
- added IC2: LM75AD,118, LM75:SOIC127P600X175-8N, symbol LM75:LM75AD,118
- TP4: value SDA1 -> OS
- TP5: value Alert -> SCL1
- TP6: value SCL1 -> SDA1
Connections:
- net Alert is gone; now on net SCL1: R7.2, TP5.1
- net GND: now also IC2.4 (GND), IC2.5 (A2), IC2.6 (A1), IC2.7 (A0)
- net SCL1: now also IC2.2 (SCL); no longer R8.2, TP6.1
- net SDA1: now also R8.2, TP6.1, IC2.1 (SDA); no longer R6.2, TP4.1
- net V_out: now also IC2.8 (VCC)
- new net OS: IC2.3 (OS), R6.2, TP4.1
Other:
- note added: "LIGHT DEPENDENT RESISTOR"
- note added: "TEMPERATURE SENSOR"
- note removed: "Connectors/Pin Headers"
- moved on the sheet: R10, R9, TP7
